Commit message: feat(sim2sim): add source rough profile and held-key RMUC control

File: src/resources/robot_descriptions/wheelbipe_V14/xacro/robot_sim.xacro (robot description, xacro)
@@ -1,7 +1,8 @@
 <?xml version="1.0"?>
 <robot xmlns:xacro="http://wiki.ros.org/xacro" name="wheelbipe_V14">
+  <xacro:arg name="sim_profile" default="deployment"/>
   <xacro:include filename="$(find robot_descriptions)/wheelbipe_V14/xacro/description.xacro"/>
   <xacro:include filename="$(find robot_descriptions)/wheelbipe_V14/xacro/ros2control.xacro"/>
   <xacro:description/>
-  <xacro:ros2control name="MujocoControl" backend="sim"/>
+  <xacro:ros2control name="MujocoControl" backend="sim" sim_profile="$(arg sim_profile)"/>
 </robot>

File: src/resources/robot_descriptions/wheelbipe_V14/xacro/ros2control.xacro (robot description, xacro)
@@ -13,5 +13,5 @@
   <xacro:property name="v14_actuator_speed_droop_per_rad_s" value="0.055"/>
   <xacro:property name="v14_actuator_min_speed_gain" value="0.55"/>
-  <xacro:macro name="ros2control" params="name backend='sim' serial_port='/dev/wheelbipe_h7' baudrate='2000000' serial_reconnect_interval_ms='1000' state_timeout_ms='100'">
+  <xacro:macro name="ros2control" params="name sim_profile='deployment' backend='sim' serial_port='/dev/wheelbipe_h7' baudrate='2000000' serial_reconnect_interval_ms='1000' state_timeout_ms='100'">
     <ros2_control name="${name}" type="system">
       <hardware>
@@ -19,10 +19,10 @@
           <plugin>mujoco_ros2_control/MujocoSystem</plugin>
           <param name="gas_spring_model_enabled">true</param>
-          <param name="gas_spring_q_min">-0.005</param>
-          <param name="gas_spring_q_max">0.07</param>
-          <param name="gas_spring_force_at_q_min">650.0</param>
-          <param name="gas_spring_force_at_q_max">450.0</param>
+          <param name="gas_spring_q_min">${-0.015 if sim_profile == 'source_v14' else -0.005}</param>
+          <param name="gas_spring_q_max">${0.06076 if sim_profile == 'source_v14' else 0.07}</param>
+          <param name="gas_spring_force_at_q_min">${616.457142857143 if sim_profile == 'source_v14' else 650.0}</param>
+          <param name="gas_spring_force_at_q_max">${400.0 if sim_profile == 'source_v14' else 450.0}</param>
           <param name="gas_spring_manual_passive_enabled">true</param>
-          <param name="gas_spring_manual_viscous_damping">500.0</param>
+          <param name="gas_spring_manual_viscous_damping">${50.0 if sim_profile == 'source_v14' else 500.0}</param>
           <param name="gas_spring_manual_static_friction">0.0</param>
           <param name="gas_spring_manual_velocity_epsilon">0.01</param>
@@ -37,5 +37,5 @@
       </hardware>
       <joint name="left_front1_joint">
-        <param name="actuator_model_enabled">${v14_actuator_model_enabled}</param>
+        <param name="actuator_model_enabled">${v14_actuator_model_enabled and sim_profile != 'source_v14'}</param>
         <param name="actuator_time_constant_s">${v14_actuator_time_constant_s}</param>
         <param name="actuator_transport_delay_s">${v14_actuator_transport_delay_s}</param>
@@ -58,5 +58,5 @@
       </joint>
       <joint name="left_rear1_joint">
-        <param name="actuator_model_enabled">${v14_actuator_model_enabled}</param>
+        <param name="actuator_model_enabled">${v14_actuator_model_enabled and sim_profile != 'source_v14'}</param>
         <param name="actuator_time_constant_s">${v14_actuator_time_constant_s}</param>
         <param name="actuator_transport_delay_s">${v14_actuator_transport_delay_s}</param>
@@ -79,5 +79,5 @@
       </joint>
       <joint name="right_front1_joint">
-        <param name="actuator_model_enabled">${v14_actuator_model_enabled}</param>
+        <param name="actuator_model_enabled">${v14_actuator_model_enabled and sim_profile != 'source_v14'}</param>
         <param name="actuator_time_constant_s">${v14_actuator_time_constant_s}</param>
         <param name="actuator_transport_delay_s">${v14_actuator_transport_delay_s}</param>
@@ -100,5 +100,5 @@
       </joint>
       <joint name="right_rear1_joint">
-        <param name="actuator_model_enabled">${v14_actuator_model_enabled}</param>
+        <param name="actuator_model_enabled">${v14_actuator_model_enabled and sim_profile != 'source_v14'}</param>
         <param name="actuator_time_constant_s">${v14_actuator_time_constant_s}</param>
         <param name="actuator_transport_delay_s">${v14_actuator_transport_delay_s}</param>
